Commit message: EM and LA_lifters now working

File: description/robot_core.xacro (robot description, xacro)
@@ -12,4 +12,11 @@
     </material>
     <link name="base_link">
+    </link>
+    <joint name="base_footprint_joint" type="fixed">
+        <parent link="base_link"/>
+        <child link="base_footprint"/>
+        <origin xyz="0 0 0" rpy="0 0 0"/>
+    </joint>
+    <link name="base_footprint">
     </link>
     <joint name="chassis_joint" type="fixed">
@@ -39,5 +46,5 @@
         <material>Gazebo/White</material>
     </gazebo>
-    <joint name="lrw_joint" type="continuous">
+    <joint name="lrw_joint" type="fixed">
         <parent link="base_link"/>
         <child link="lrw_link"/>
@@ -69,5 +76,5 @@
         <fdir1 value="1 0 0"/>
     </gazebo>
-    <joint name="rrw_joint" type="continuous">
+    <joint name="rrw_joint" type="fixed">
         <parent link="base_link"/>
         <child link="rrw_link"/>
@@ -99,5 +106,5 @@
         <fdir1 value="1 0 0"/>
     </gazebo>
-    <joint name="lfw_joint" type="continuous">
+    <joint name="lfw_joint" type="fixed">
         <parent link="base_link"/>
         <child link="lfw_link"/>
@@ -129,5 +136,5 @@
         <fdir1 value="1 0 0"/>
     </gazebo>
-    <joint name="rfw_joint" type="continuous">
+    <joint name="rfw_joint" type="fixed">
         <parent link="base_link"/>
         <child link="rfw_link"/>

File: description/wcs.urdf.xacro (robot description, xacro)
@@ -2,6 +2,6 @@
 <robot xmlns:xacro="http://www.ros.org/wiki/xacro" name="wheelchock_robot">
     <xacro:include filename="robot_core.xacro"/>
-    <xacro:include filename="ros2_control.xacro"/>
     <xacro:include filename="lidar.xacro"/>
     <xacro:include filename="depth_camera.xacro"/>
+    <xacro:include filename="imu.xacro"/>
 </robot>
